Commit message: it works fine with abb robot from tutorial

File: urdf/kr300r2500ultra.xacro (robot description, xacro)
@@ -1,6 +1,6 @@
 <?xml version="1.0"?>
-<robot name="kuka_kr120r2500pro" xmlns:xacro="http://wiki.ros.org/xacro">
-    <xacro:include filename="$(find practice)/urdf/kr120r2500pro_macro.xacro" />
-    <xacro:kuka_kr120r2500pro prefix=""/>
+<robot name="kuka_kr300r2500ultra" xmlns:xacro="http://wiki.ros.org/xacro">
+    <xacro:include filename="$(find practice)/urdf/kr300r2500ultra_macro.xacro" />
+    <xacro:kuka_kr300r2500ultra prefix=""/>
     <link name="world"/>
     <joint name="world__base_link" type="fixed">
@@ -9,4 +9,5 @@
         <origin xyz="0 0 0" rpy="0 0 0"/>
     </joint>
+<!--
     <link name="box">
         <visual>
@@ -26,3 +27,4 @@
         <origin xyz="2 0.25 1" rpy="0 0 0"/>
     </joint>
+-->
 </robot>

File: urdf/kr300r2500ultra_macro.xacro (robot description, xacro)
@@ -2,5 +2,5 @@
 <robot xmlns:xacro="http://wiki.ros.org/xacro">
   <xacro:property name="DEG2RAD" value="0.017453292519943295"/>
-  <xacro:macro name="kuka_kr120r2500pro" params="prefix">
+  <xacro:macro name="kuka_kr300r2500ultra" params="prefix">
     <!-- LINKS -->
     <!-- base link -->
